Commit message: green ball resized, move based disabled for one of the robots in two robots launch

File: py3dx_gazebo/xacro/ball/ball.xacro (robot description, xacro)
@@ -18,5 +18,5 @@
       <origin xyz="0 0 0" rpy="0 1.57 0"/>
       <geometry>
-        <sphere radius="0.03"/>
+        <sphere radius="0.2"/>
       </geometry>
       <material name="green"/>
@@ -25,5 +25,5 @@
       <origin xyz="0 0 0" rpy="0 1.57 0"/>
       <geometry>
-        <sphere radius="0.03"/>
+        <sphere radius="0.2"/>
       </geometry>
     </collision>
